File: KiCad-Power_Board.kicad_pcb (KiCad board)
At the start: 2 copper layers, 24 parts, among them P1 Batt, P10 Batt, P11 Switch, P12 Out, P2 Switch, P3 Out, P4 Batt, P5 Switch, P6 Out, P7 Batt, P8 Switch, P9 Out, U1 LM3480-3.3, U2 LM3480-3.3, U3 LM3480-3.3, U4 LM3480-3.3

Commit message: misc
Parts:
- added I1: ACS758, KiCad-Dev:ACS758-hall, F.Cu at (251.5, 89.7)
- added P13: CONN_01X02, Pin_Headers:Pin_Header_Straight_1x02, F.Cu at (213.9, 70.9)
- added P14, P15, P16: CONN_01X02, Pin_Headers:Pin_Header_Straight_1x02, F.Cu at (241.3, 115.1)
Routing:
- net GND: track 90.7 -> 199.8 mm
- net Net-(D1-Pad2): track 3.35 -> 7.26 mm
- net Net-(F1-Pad2): track 30.2 -> 31.6 mm

Commit message: test
Parts:
- removed I1: ACS758, KiCad-Dev:ACS758-hall
- removed P11, P5, P8: Switch, KiCad-Dev:XT60
- removed P13, P14, P15, P16: CONN_01X02, Pin_Headers:Pin_Header_Straight_1x02
- added U5: ACS758, KiCad-Dev:ACS758_Vertical, F.Cu at (228.6, 66.0)
- added U6: ACS758, KiCad-Dev:ACS758_Vertical, F.Cu at (228.6, 55.9)
- added U7: ACS758, KiCad-Dev:ACS758_Vertical, F.Cu at (228.6, 86.4)
- added U8: ACS758, KiCad-Dev:ACS758_Vertical, F.Cu at (228.6, 76.2)
- P2: value Switch -> PWR_Status; footprint KiCad-Dev:XT60 -> Pin_Headers:Pin_Header_Straight_1x06
- moved P2 94.0 mm to (261.6, 63.5)
- moved P6 46.6 mm to (251.3, 55.9)
- moved P4 43.4 mm to (165.2, 55.9)
- moved U2 40.7 mm to (213.4, 55.9)
- moved D2 40.6 mm to (208.3, 55.9)
- moved F2 40.6 mm to (193.0, 55.9)
- moved P12 22.9 mm to (251.5, 76.2)
- moved P3 22.9 mm to (251.5, 66.0)
- moved P9 22.9 mm to (251.3, 86.4)
- moved P1 15.2 mm to (165.2, 66.0)
- moved P10 15.2 mm to (165.2, 86.4)
- moved P7 15.2 mm to (165.2, 76.2)
- moved U1 1.27 mm to (213.4, 66.0)
- moved U3 1.27 mm to (213.4, 86.4)
- moved U4 1.27 mm to (213.4, 76.2)
Connections:
- D1 pad 2: Net-(D1-Pad2) -> /pwr_module2/PWR_3.3V_Status
- D2 pad 2: Net-(D2-Pad2) -> /pwr_module1/PWR_3.3V_Status
- D3 pad 2: Net-(D3-Pad2) -> /pwr_module4/PWR_3.3V_Status
- D4 pad 2: Net-(D4-Pad2) -> /pwr_module3/PWR_3.3V_Status
- F1 pad 1: Net-(F1-Pad1) -> +BATT
- F2 pad 1: Net-(F2-Pad1) -> +BATT
- F3 pad 1: Net-(F3-Pad1) -> +BATT
- F4 pad 1: Net-(F4-Pad1) -> +BATT
- P12 pad 2: Net-(F4-Pad2) -> Net-(P12-Pad2)
- P2 pad 1: +BATT -> /pwr_module1/PWR_3.3V_Status
- P2 pad 2: Net-(F1-Pad1) -> /pwr_module2/PWR_3.3V_Status
- P3 pad 2: Net-(F1-Pad2) -> Net-(P3-Pad2)
- P6 pad 2: Net-(F2-Pad2) -> Net-(P6-Pad2)
- P9 pad 2: Net-(F3-Pad2) -> Net-(P9-Pad2)
- U1 pad 1: Net-(D1-Pad2) -> /pwr_module2/PWR_3.3V_Status
- U2 pad 1: Net-(D2-Pad2) -> /pwr_module1/PWR_3.3V_Status
- U3 pad 1: Net-(D3-Pad2) -> /pwr_module4/PWR_3.3V_Status
- U4 pad 1: Net-(D4-Pad2) -> /pwr_module3/PWR_3.3V_Status
Routing:
- net (no net): track 0.00 -> 76.2 mm
- net /pwr_module4/PWR_3.3V_Status: track 0.00 -> 70.7 mm
- net /pwr_module3/PWR_3.3V_Status: track 0.00 -> 63.1 mm
- net /pwr_module1/PWR_3.3V_Status: track 0.00 -> 57.4 mm
- net /pwr_module2/PWR_3.3V_Status: track 0.00 -> 57.1 mm
- net +BATT: track 61.0 -> 81.3 mm
- net Net-(F4-Pad1): track 14.9 -> 0.00 mm
- net Net-(F3-Pad1): track 14.9 -> 0.00 mm
- net Net-(F1-Pad1): track 14.9 -> 0.00 mm
- net GND: track 199.8 -> 184.9 mm
- net Net-(F2-Pad1): track 14.8 -> 0.00 mm
- net Net-(P3-Pad2): track 0.00 -> 10.3 mm
- net Net-(P12-Pad2): track 0.00 -> 10.3 mm
- net Net-(P9-Pad2): track 0.00 -> 10.2 mm
- net Net-(P6-Pad2): track 0.00 -> 10.2 mm
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Other:
- board outline added: 121.9 x 61 mm
- board text added: "Battery"
- board text added: "Fused Out"

Commit message: test
Parts:
- added I1: ACS758, KiCad-Dev:ACS758-hall, F.Cu at (273.1, 77.5)
Routing:
- net GND: track 184.9 -> 361.8 mm
- net /pwr_module4/PWR_3.3V_Status: track 70.7 -> 71.9 mm
- net /pwr_module3/PWR_3.3V_Status: track 63.1 -> 63.9 mm
- net /pwr_module2/PWR_3.3V_Status: track 57.1 -> 57.8 mm
